File: schematics/LampenSteuerung PWM.brd (EAGLE design)
At the start: 41.2 x 33.8 mm, 47 parts, among them IC1 LM358D, IC2 TSOP34836, IC4 TS2951-3.0, Q1 BCR135, Q2 BCR135, Q3 BCR135, T1 SFH320, T2 IRLML6346, X2 MKDSN1,5/5-5,08

Commit message: added driver and encoder pcb
Parts:
- added D2: 27V, diode:SMBJ
Connections:
- net GND: now also D2.A
- net N$9: now also D2.C
Changed lines of the file:
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@@
 <?xml version="1.0" encoding="utf-8"?>
 <!DOCTYPE eagle SYSTEM "eagle.dtd">
-<eagle version="7.0.0">
+<eagle version="7.5.0">
 <drawing>
 <settings>
@@
 <attribute name="OC_FARNELL" value="unknown" x="38.354" y="27.686" size="1.778" layer="28" rot="MR180" display="off"/>
 </element>
+<element name="D2" library="diode" package="SMBJ" value="27V" x="-2.413" y="-15.367"/>
 </elements>
 <signals>
@@
 <contactref element="T1" pad="C"/>
 <contactref element="T2" pad="2"/>
+<contactref element="D2" pad="A"/>
+<wire x1="37.084" y1="23.053" x2="40.894" y2="20.574" width="0" layer="19" extent="16-16"/>
+<wire x1="37.846" y1="24.376" x2="37.084" y2="23.053" width="0" layer="19" extent="1-16"/>
+<wire x1="34.925" y1="23.368" x2="37.084" y2="23.053" width="0" layer="19" extent="16-16"/>
+<wire x1="37.4142" y1="26.67" x2="37.846" y2="24.376" width="0" layer="19" extent="1-16"/>
+<wire x1="35.687" y1="27.305" x2="37.4142" y2="26.67" width="0" layer="19" extent="16-16"/>
+<wire x1="33.531" y1="25.273" x2="34.925" y2="23.368" width="0" layer="19" extent="16-16"/>
+<wire x1="27.686" y1="22.352" x2="33.531" y2="25.273" width="0" layer="19" extent="16-16"/>
+<wire x1="25.467" y1="22.987" x2="27.686" y2="22.352" width="0" layer="19" extent="16-16"/>
+<wire x1="26.709" y1="25.273" x2="25.467" y2="22.987" width="0" layer="19" extent="16-16"/>
+<wire x1="22.86" y1="22.413" x2="25.467" y2="22.987" width="0" layer="19" extent="16-16"/>
+<wire x1="22.86" y1="24.13" x2="22.86" y2="22.413" width="0" layer="19" extent="16-16"/>
+<wire x1="27.686" y1="19.685" x2="27.686" y2="22.352" width="0" layer="19" extent="1-1"/>
+<wire x1="27.1991" y1="29.312" x2="26.709" y2="25.273" width="0" layer="19" extent="16-16"/>
+<wire x1="27.305" y1="14.478" x2="27.686" y2="19.685" width="0" layer="19" extent="1-1"/>
+<wire x1="25.527" y1="14.439" x2="27.305" y2="14.478" width="0" layer="19" extent="16-16"/>
+<wire x1="25.2762" y1="13.152" x2="25.527" y2="14.439" width="0" layer="19" extent="1-16"/>
+<wire x1="27.051" y1="10.414" x2="25.2762" y2="13.152" width="0" layer="19" extent="1-1"/>
+<wire x1="22.225" y1="17.145" x2="25.527" y2="14.439" width="0" layer="19" extent="16-16"/>
+<wire x1="18.753" y1="19.111" x2="22.225" y2="17.145" width="0" layer="19" extent="1-1"/>
+<wire x1="18.88" y1="14.666" x2="22.225" y2="17.145" width="0" layer="19" extent="1-1"/>
+<wire x1="16.129" y1="14.163" x2="18.88" y2="14.666" width="0" layer="19" extent="1-16"/>
+<wire x1="16.764" y1="11.557" x2="16.129" y2="14.163" width="0" layer="19" extent="16-16"/>
+<wire x1="18.88" y1="10.475" x2="16.764" y2="11.557" width="0" layer="19" extent="1-1"/>
+<wire x1="20.955" y1="11.557" x2="18.88" y2="10.475" width="0" layer="19" extent="1-1"/>
+<wire x1="17.399" y1="23.583" x2="18.753" y2="19.111" width="0" layer="19" extent="1-16"/>
+<wire x1="14.478" y1="22.793" x2="17.399" y2="23.583" width="0" layer="19" extent="16-16"/>
+<wire x1="11" y1="22.225" x2="14.478" y2="22.793" width="0" layer="19" extent="1-16"/>
+<wire x1="12.7" y1="19.558" x2="11" y2="22.225" width="0" layer="19" extent="1-1"/>
+<wire x1="9.017" y1="17.995" x2="12.7" y2="19.558" width="0" layer="19" extent="16-16"/>
+<wire x1="6.604" y1="17.78" x2="9.017" y2="17.995" width="0" layer="19" extent="16-16"/>
+<wire x1="6.604" y1="19.624" x2="6.604" y2="17.78" width="0" layer="19" extent="16-16"/>
+<wire x1="18.415" y1="5.461" x2="18.88" y2="10.475" width="0" layer="19" extent="1-1"/>
+<wire x1="18.415" y1="2.921" x2="18.415" y2="5.461" width="0" layer="19" extent="1-1"/>
+<wire x1="12.231" y1="8.382" x2="16.764" y2="11.557" width="0" layer="19" extent="16-16"/>
+<wire x1="11.469" y1="5.461" x2="12.231" y2="8.382" width="0" layer="19" extent="1-16"/>
+<wire x1="9.144" y1="5.588" x2="11.469" y2="5.461" width="0" layer="19" extent="1-1"/>
+<wire x1="12.7" y1="2.921" x2="11.469" y2="5.461" width="0" layer="19" extent="1-1"/>
+<wire x1="11.9591" y1="29.312" x2="14.478" y2="22.793" width="0" layer="19" extent="16-16"/>
+<wire x1="30.861" y1="3.048" x2="27.051" y2="10.414" width="0" layer="19" extent="1-1"/>
+<wire x1="37.426" y1="7.874" x2="30.861" y2="3.048" width="0" layer="19" extent="1-1"/>
+<wire x1="39.878" y1="7.874" x2="37.426" y2="7.874" width="0" layer="19" extent="1-1"/>
+<wire x1="-0.373" y1="-15.367" x2="12.7" y2="2.921" width="0" layer="19" extent="1-1"/>
 </signal>
 <signal name="+UB">
@@
 <wire x1="38.354" y1="29.845" x2="38.354" y2="28.7274" width="0.4064" layer="16"/>
 <wire x1="38.354" y1="28.7274" x2="38.3794" y2="28.702" width="0.4064" layer="16"/>
+<contactref element="D2" pad="C"/>
+<wire x1="-4.443" y1="-15.367" x2="12.761" y2="26.162" width="0" layer="19" extent="1-16"/>
 </signal>
 <signal name="N$21">
