File: schematics/LampenSteuerung PWM.sch (EAGLE design)
At the start: 47 parts, among them IC1 LM358D, IC2 TSOP34836, IC4 TS2951-3.0, Q1 BCR135, Q2 BCR135, Q3 BCR135, T1 SFH320, T2 IRLML6346, X2 MKDSN1,5/5-5,08

Commit message: added driver and encoder pcb
Parts:
- added D2: 27V, diode:SUPPRESSOR-SMBJ
Connections:
- net GND: now also D2.A
- net N$9: now also D2.C
Changed lines of the file:
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@@
 <?xml version="1.0" encoding="utf-8"?>
 <!DOCTYPE eagle SYSTEM "eagle.dtd">
-<eagle version="7.0.0">
+<eagle version="7.5.0">
 <drawing>
 <settings>
@@
 <part name="SUPPLY5" library="supply2" deviceset="+UB" device=""/>
 <part name="T2" library="zetex" deviceset="NMOSSOT23" device="" value="IRLML6346"/>
+<part name="D2" library="diode" deviceset="SUPPRESSOR-" device="SMBJ" value="27V"/>
 </parts>
 <sheets>
@@
 <instance part="SUPPLY5" gate="G$1" x="71.12" y="134.62"/>
 <instance part="T2" gate="A" x="147.32" y="-17.78"/>
+<instance part="D2" gate="G$1" x="154.94" y="-27.94"/>
 </instances>
 <busses>
@@
 <wire x1="160.02" y1="-12.7" x2="162.56" y2="-12.7" width="0.1524" layer="91"/>
 <wire x1="147.32" y1="-22.86" x2="147.32" y2="-40.64" width="0.1524" layer="91"/>
-<wire x1="147.32" y1="-40.64" x2="160.02" y2="-40.64" width="0.1524" layer="91"/>
+<wire x1="147.32" y1="-40.64" x2="154.94" y2="-40.64" width="0.1524" layer="91"/>
 <pinref part="R19" gate="G$1" pin="1"/>
+<wire x1="154.94" y1="-40.64" x2="160.02" y2="-40.64" width="0.1524" layer="91"/>
 <wire x1="139.7" y1="-35.56" x2="139.7" y2="-40.64" width="0.1524" layer="91"/>
 <wire x1="139.7" y1="-40.64" x2="147.32" y2="-40.64" width="0.1524" layer="91"/>
@@
 <junction x="160.02" y="-40.64"/>
 <pinref part="T2" gate="A" pin="S"/>
+<pinref part="D2" gate="G$1" pin="A"/>
+<wire x1="154.94" y1="-30.48" x2="154.94" y2="-40.64" width="0.1524" layer="91"/>
+<junction x="154.94" y="-40.64"/>
 </segment>
 <segment>
@@
 <pinref part="X2" gate="-4" pin="KL"/>
 <pinref part="R4" gate="G$1" pin="2"/>
-<wire x1="162.56" y1="-7.62" x2="147.32" y2="-7.62" width="0.1524" layer="91"/>
+<wire x1="162.56" y1="-7.62" x2="154.94" y2="-7.62" width="0.1524" layer="91"/>
+<wire x1="154.94" y1="-7.62" x2="147.32" y2="-7.62" width="0.1524" layer="91"/>
 <wire x1="147.32" y1="-7.62" x2="137.16" y2="-7.62" width="0.1524" layer="91"/>
 <wire x1="147.32" y1="-12.7" x2="147.32" y2="-7.62" width="0.1524" layer="91"/>
@@
 <wire x1="147.32" y1="-7.62" x2="147.32" y2="-2.54" width="0.1524" layer="91"/>
 <pinref part="T2" gate="A" pin="D"/>
-</segment>
-</net>
+<pinref part="D2" gate="G$1" pin="C"/>
+<wire x1="154.94" y1="-25.4" x2="154.94" y2="-7.62" width="0.1524" layer="91"/>
+<junction x="154.94" y="-7.62"/>
+</segment>
+</net>
